Commit message: 解决Gazebo启动模型崩溃问题

File: description/robot.urdf.xacro (robot description, xacro)
@@ -2,3 +2,4 @@
 <robot xmlns:xacro="http://www.ros.org/wiki/xacro" name="Articubot_CT">
     <xacro:include filename="robot_core.xacro" />
+    <xacro:include filename="gazebo_control.xacro" />
 </robot>

File: description/robot_core.xacro (robot description, xacro)
@@ -1,5 +1,5 @@
 <?xml version="1.0"?>
 <xacro:robot xmlns:xacro="http://www.ros.org/wiki/xacro">
-    <xacro:include filename="$(find Articubot_CT)/description/inertial_macros.xacro"/>
+    <xacro:include filename="inertial_macros.xacro"/>
     <material name="white">
         <color rgba="1 1 1 1" />
@@ -74,4 +74,7 @@
         <xacro:chassis_inertial mass="0.5" x="0.3" y="0.3" z="0.15"/>
     </link>
+    <gazebo reference="chassis">
+        <material>Gazebo/White</material>
+    </gazebo>
     <!-- LEFT WHEEL LINK -->
     <joint name="left_wheel_joint" type="continuous">
@@ -80,4 +83,5 @@
         <origin xyz="0 0.175 0" rpy="-$(eval pi/2) 0 0"/>
         <axis xyz="0 0 1"/>
+        <limit effort="10.0" velocity="10.0"/>
     </joint>
     <link name="left_wheel">
@@ -94,5 +98,9 @@
         </collision>
         <xacro:wheel_inertial mass="0.1" length="0.04" radius="0.05"/>
+            <origin xyz="0 0 0" rpy="0 0 0"/>
     </link>
+    <gazebo reference="left_wheel">
+        <material>Gazebo/Blue</material>
+    </gazebo>
     <!-- RIGHT WHEEL LINK -->
     <joint name="right_wheel_joint" type="continuous">
@@ -101,4 +109,5 @@
         <origin xyz="0 -0.175 0" rpy="$(eval pi/2) 0 0"/>
         <axis xyz="0 0 -1"/>
+        <limit effort="10.0" velocity="10.0"/>
     </joint>
     <link name="right_wheel">
@@ -115,5 +124,9 @@
         </collision>
         <xacro:wheel_inertial mass="0.1" length="0.04" radius="0.05"/>
+            <origin xyz="0 0 0" rpy="0 0 0"/>
     </link>
+    <gazebo reference="right_wheel">
+        <material>Gazebo/Blue</material>
+    </gazebo>
     <!-- CASTER WHEEL LINK -->
     <joint name="caster_wheel_joint" type="fixed">
@@ -135,4 +148,10 @@
         </collision>
         <xacro:caster_wheel_inertial mass="0.1" radius="0.05"/>
+            <origin xyz="0 0 0" rpy="0 0 0"/>
     </link>
+    <gazebo reference="caster_wheel">
+        <material>Gazebo/Black</material>
+        <mu1 value="0.001"/>
+        <mu2 value="0.001"/>
+    </gazebo>
 </xacro:robot>
