Commit message: Rviz2 Model odom  fix

File: description/gazebo_control.xacro (robot description, xacro)
@@ -1,4 +1,25 @@
 <?xml version="1.0"?>
 <robot xmlns:xacro="http://www.ros.org/wiki/xacro" >
+<!-- 差速驱动插件 -->
+        <gazebo>
+            <plugin name="gz::sim::systems::DiffDrive" filename="libgz-sim-diff-drive-system.so">
+                <left_joint>left_wheel_joint</left_joint>
+                <right_joint>right_wheel_joint</right_joint>
+                <wheel_separation>0.35</wheel_separation>
+                <wheel_radius>0.05</wheel_radius>
+                <max_wheel_torque>200</max_wheel_torque>
+                <max_wheel_acceleration>10.0</max_wheel_acceleration>
+                <odometry_frame>odom</odometry_frame>
+                <robot_base_frame>base_link</robot_base_frame>
+                <publish_odom>true</publish_odom>
+                <publish_odom_tf>true</publish_odom_tf>
+                <publish_wheel_tf>true</publish_wheel_tf>
+                <left_joint_parent>base_link</left_joint_parent>
+                <right_joint_parent>base_link</right_joint_parent>
+                <topic>/cmd_vel</topic>
+                <odom_topic>/model/Articubot_CT/odometry</odom_topic>
+                <odom_frame>odom</odom_frame>
+                <enable_covariance>true</enable_covariance>
+            </plugin>
         <!-- 驱动轮关节 -->
         <gazebo reference="left_wheel">
@@ -24,22 +45,4 @@
             </ode>
         </gazebo>
-        <!-- 差速驱动插件 -->
-        <gazebo>
-            <plugin name="gz::sim::systems::DiffDrive" filename="libgz-sim-diff-drive-system.so">
-                <robot_base_frame>base_link</robot_base_frame>
-                <left_joint>left_wheel_joint</left_joint>
-                <right_joint>right_wheel_joint</right_joint>
-                <wheel_separation>0.35</wheel_separation>
-                <wheel_radius>0.05</wheel_radius>
-                <left_joint_parent>base_link</left_joint_parent>
-                <right_joint_parent>base_link</right_joint_parent>
-                <topic>/cmd_vel</topic>
-                <odom_topic>/model/Articubot_CT/odometry</odom_topic>
-                <odom_frame>odom</odom_frame>
-                <publish_odom>true</publish_odom>
-                <publish_wheel_tf>false</publish_wheel_tf>
-                <publish_odom_tf>false</publish_odom_tf>
-                <enable_covariance>true</enable_covariance>
-            </plugin>
             <!-- 关节状态发布插件 -->
             <plugin name="gz::sim::systems::JointStatePublisher" filename="libgz-sim-joint-state-publisher-system.so">

File: description/robot_core.xacro (robot description, xacro)
@@ -14,5 +14,5 @@
         <color rgba="0 0 0 1"/>
     </material>
-    <!-- 添加 dummy link 作为根节点
+    <!-- 添加 dummy link 作为根节点 -->
     <link name="world_link">
         <visual>
@@ -27,28 +27,28 @@
             </geometry>
         </collision>
-    </link> -->
-    <!-- 固定关节连接 world_link 和 base_link
+    </link>
+    <!-- 固定关节连接 world_link 和 base_link -->
     <joint name="world_joint" type="fixed">
         <parent link="world_link"/>
         <child link="base_link"/>
         <origin xyz="0 0 0"/>
-    </joint> -->
+    </joint>
     <!-- 原始 base_link -->
     <link name="base_link">
-        <!-- <visual>
+        <visual>
             <geometry>
-                <box size="0.5 0.3 0.2"/>
+                <box size="0.001 0.001 0.001"/>
             </geometry>
-            <material name="white"/>
+            <material name="black"/>
         </visual>
         <collision>
             <geometry>
-                <box size="0.5 0.6 0.2"/>
+                <box size="0.001 0.001 0.001"/>
             </geometry>
         </collision>
         <inertial>
-            <mass value="1.0"/>
-            <inertia ixx="0.1" ixy="0.0" ixz="0.0" iyy="0.1" iyz="0.0" izz="0.1"/>
-        </inertial> -->
+            <mass value="0.01"/>
+            <inertia ixx="0.0001" ixy="0.0" ixz="0.0" iyy="0.0001" iyz="0.0" izz="0.0001"/>
+        </inertial>
     </link>
     <joint name="chassis_joint" type="fixed">
@@ -98,5 +98,4 @@
         </collision>
         <xacro:wheel_inertial mass="0.1" length="0.04" radius="0.05"/>
-            <origin xyz="0 0 0" rpy="0 0 0"/>
     </link>
     <gazebo reference="left_wheel">
@@ -124,5 +123,4 @@
         </collision>
         <xacro:wheel_inertial mass="0.1" length="0.04" radius="0.05"/>
-            <origin xyz="0 0 0" rpy="0 0 0"/>
     </link>
     <gazebo reference="right_wheel">
@@ -148,5 +146,4 @@
         </collision>
         <xacro:caster_wheel_inertial mass="0.1" radius="0.05"/>
-            <origin xyz="0 0 0" rpy="0 0 0"/>
     </link>
     <gazebo reference="caster_wheel">

Commit message: Rviz2 Model odom fix

File: description/gazebo_control.xacro (robot description, xacro)
@@ -1,52 +1,55 @@
 <?xml version="1.0"?>
-<robot xmlns:xacro="http://www.ros.org/wiki/xacro" >
-<!-- 差速驱动插件 -->
-        <gazebo>
-            <plugin name="gz::sim::systems::DiffDrive" filename="libgz-sim-diff-drive-system.so">
-                <left_joint>left_wheel_joint</left_joint>
-                <right_joint>right_wheel_joint</right_joint>
-                <wheel_separation>0.35</wheel_separation>
-                <wheel_radius>0.05</wheel_radius>
-                <max_wheel_torque>200</max_wheel_torque>
-                <max_wheel_acceleration>10.0</max_wheel_acceleration>
-                <odometry_frame>odom</odometry_frame>
-                <robot_base_frame>base_link</robot_base_frame>
-                <publish_odom>true</publish_odom>
-                <publish_odom_tf>true</publish_odom_tf>
-                <publish_wheel_tf>true</publish_wheel_tf>
-                <left_joint_parent>base_link</left_joint_parent>
-                <right_joint_parent>base_link</right_joint_parent>
-                <topic>/cmd_vel</topic>
-                <odom_topic>/model/Articubot_CT/odometry</odom_topic>
-                <odom_frame>odom</odom_frame>
-                <enable_covariance>true</enable_covariance>
-            </plugin>
-        <!-- 驱动轮关节 -->
-        <gazebo reference="left_wheel">
-            <mu1>1.0</mu1>
-            <mu2>1.0</mu2>
-            <material>Gazebo/Blue</material>
-            <ode>
-                <kp>10000000.0</kp>
-                <kd>1.0</kd>
-                <minDepth>0.001</minDepth>
-                <maxVel>10.0</maxVel>
-            </ode>
-        </gazebo>
-        <gazebo reference="right_wheel">
-            <mu1>1.0</mu1>
-            <mu2>1.0</mu2>
-            <material>Gazebo/Blue</material>
-            <ode>
-                <kp>10000000.0</kp>
-                <kd>1.0</kd>
-                <minDepth>0.001</minDepth>
-                <maxVel>10.0</maxVel>
-            </ode>
-        </gazebo>
-            <!-- 关节状态发布插件 -->
-            <plugin name="gz::sim::systems::JointStatePublisher" filename="libgz-sim-joint-state-publisher-system.so">
-                <update_rate>50</update_rate>
-            </plugin>
-        </gazebo>
+<robot xmlns:xacro="http://www.ros.org/wiki/xacro">
+    <!-- 差速驱动插件 -->
+    <gazebo>
+        <plugin name="gz::sim::systems::DiffDrive" filename="libgz-sim-diff-drive-system.so">
+            <left_joint>left_wheel_joint</left_joint>
+            <right_joint>right_wheel_joint</right_joint>
+            <wheel_separation>0.35</wheel_separation>
+            <wheel_radius>0.05</wheel_radius>
+            <max_wheel_torque>200</max_wheel_torque>
+            <max_wheel_acceleration>10.0</max_wheel_acceleration>
+            <odometry_frame>odom</odometry_frame>
+            <robot_base_frame>base_link</robot_base_frame>
+            <publish_odom>true</publish_odom>
+            <publish_odom_tf>true</publish_odom_tf>
+            <publish_wheel_tf>true</publish_wheel_tf>
+            <left_joint_parent>base_link</left_joint_parent>
+            <right_joint_parent>base_link</right_joint_parent>
+            <topic>/cmd_vel</topic>
+            <odom_topic>/model/Articubot_CT/odometry</odom_topic>
+            <odom_frame>odom</odom_frame>
+            <enable_covariance>true</enable_covariance>
+        </plugin>
+    </gazebo>
+    <!-- 驱动轮属性 -->
+    <gazebo reference="left_wheel">
+        <mu1>1.0</mu1>
+        <mu2>1.0</mu2>
+        <material>Gazebo/Blue</material>
+        <ode>
+            <kp>10000000.0</kp>
+            <kd>1.0</kd>
+            <minDepth>0.001</minDepth>
+            <maxVel>10.0</maxVel>
+        </ode>
+    </gazebo>
+    <gazebo reference="right_wheel">
+        <mu1>1.0</mu1>
+        <mu2>1.0</mu2>
+        <material>Gazebo/Blue</material>
+        <ode>
+            <kp>10000000.0</kp>
+            <kd>1.0</kd>
+            <minDepth>0.001</minDepth>
+            <maxVel>10.0</maxVel>
+        </ode>
+    </gazebo>
+    <!-- 关节状态发布插件（必须） -->
+    <gazebo>
+        <plugin name="gz::sim::systems::JointStatePublisher" filename="libgz-sim-joint-state-publisher-system.so">
+            <update_rate>50</update_rate>
+            <topic>/model/Articubot_CT/joint_state</topic>   <!-- 明确指定话题，与桥接器匹配 -->
+        </plugin>
+    </gazebo>
 </robot>
